File: usb-atx-ctrl-redux.kicad_pcb (KiCad board)
At the start: 2 copper layers, 24.2 x 48.9 mm, 16 parts, among them J1 Amphenol 54602-908LF, SW1 SX A08, SW2 SX A08, U1 AQW210EHA, U2 AQW210EHA

Commit message: Add labels
Other:
- board text added: "BTN_PWR+"
- board text added: "BTN_PWR-"
- board text added: "BTN_RST+"
- board text added: "BTN_RST-"
- board text added: "HDD"
- board text added: "JLCJLCJLCJLC"
- board text added: "LED_HDD+"
- board text added: "LED_HDD-"
- board text added: "LED_PWR+"
- board text added: "LED_PWR-"
- board text added: "POWER"
- board text added: "POWER ON"
- board text added: "RESET"
- board text added: "usb-atx-ctrl redux Rev 0.1 (c) 2023 vmachinist"
